File: discrete555.kicad_pcb (KiCad board)
At the start: 4 copper layers, 7.6 x 10.2 mm, 44 parts, among them J1 DIP-8, Q1 CET3904E, Q10 CET3906E, Q11 CET3906E, Q12 CET3906E, Q13 CET3906E, Q14 CET3904E, Q15 CET3904E, Q16 CET3904E, Q17 CET3904E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

Commit message: Fussed with top placement a bit more
Parts:
- moved R17 0.90 mm to (44.1, 42.1), turned to 180 degrees
- moved Q25 0.40 mm to (43.0, 41.1)
- moved R16 0.25 mm to (41.8, 42.2)
- moved R9 0.23 mm to (40.4, 43.1)
- moved R10 0.19 mm to (40.6, 39.5)
- moved R6 0.19 mm to (42.2, 45.5)
Routing:
- net ~RST: track 14.2 -> 13.2 mm
- net Net-(Q25-Pad1): track 0.79 -> 1.55 mm
- net Net-(Q14-Pad1): track 1.83 -> 2.53 mm

Commit message: Added divot indicator, gotta have a divot indicator
Other:
- outline, holes or cut-outs redrawn
